File: eagle-design/schematics.sch (EAGLE design)
At the start: 17 parts, among them J1 61300411121, J2 10103594

Commit message: version 1 schematics complete
Parts:
- added C3: 100nF, resistor:C-EUC0805
- added U1: ATMEGA328P-AU, ATMEGA328P-AU:ATMEGA328P-AU
Connections:
- new net N$4: C3.2, U1.AREF
- net 5V: now also U1.AVCC, U1.VCC
- net D2: now also U1.PD2
- net D3: now also U1.PD3
- net D4: now also U1.PD4
- net D5: now also U1.PD5
- net D6: now also U1.PD6
- net GND: now also C3.1, U1.GND
- net RESET: now also U1.PC6/!RESET
- net RX: now also U1.PD0
- net SCL: now also U1.PC5
- net SDA: now also U1.PC4
- net TOSC1: now also U1.PB6
- net TOSC2: now also U1.PB7
- net TX: now also U1.PD1
Other:
- note added: "Micro-controller"
- moved on the sheet: J1, POWER_LED, R1, R2, UNLOCK_LED
