File: eagle-design/design.brd (EAGLE design)
At the start: 83.8 x 51.7 mm, 19 parts, among them J1 61300411121, J2 10103594, U1 ATMEGA328P-AU

Commit message: Fixed errors
Connections:
- net GND: now also J2.6, J2.7
Routing:
- net GND: track 208.4 -> 215.4 mm
Changed lines of the file:
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@@
 <drawing>
 <settings>
-<setting alwaysvectorfont="yes"/>
+<setting alwaysvectorfont="no"/>
 <setting verticaltext="up"/>
 </settings>
@@
 <contactref element="U1" pad="21"/>
 <wire x1="17.8714" y1="3.4544" x2="17.8714" y2="7.2644" width="0.4572" layer="1"/>
-<wire x1="7.7064" y1="8.5344" x2="11.2014" y2="8.5344" width="0.4572" layer="1"/>
-<wire x1="11.2014" y1="8.5344" x2="12.3564" y2="7.3794" width="0.4572" layer="1"/>
+<wire x1="11.2014" y1="8.5344" x2="12.4714" y2="7.2644" width="0.4572" layer="1"/>
 <wire x1="12.4714" y1="7.2644" x2="17.8714" y2="7.2644" width="0.4572" layer="1"/>
 <wire x1="37.3814" y1="10.6744" x2="13.3414" y2="10.6744" width="0.4572" layer="1"/>
@@
 <wire x1="17.5514" y1="12.9794" x2="17.5514" y2="9.1694" width="0.4572" layer="16"/>
 <wire x1="35.3822" y1="28.8036" x2="40.6314" y2="28.8036" width="0.4572" layer="1"/>
-<contactref element="J2" pad="SH1"/>
-<contactref element="J2" pad="SH4"/>
-<contactref element="J2" pad="SH3"/>
-<contactref element="J2" pad="SH2"/>
-<contactref element="J2" pad="5"/>
-<wire x1="4.8514" y1="12.5294" x2="5.3522" y2="13.0302" width="0.4572" layer="1"/>
-<wire x1="5.3522" y1="13.0302" x2="5.9436" y2="13.0302" width="0.4572" layer="1"/>
-<wire x1="4.8514" y1="12.5294" x2="4.8514" y2="18.6944" width="0.4572" layer="1"/>
-<wire x1="4.8514" y1="18.6944" x2="5.4864" y2="19.3294" width="0.4572" layer="1"/>
-<wire x1="7.8814" y1="12.2294" x2="7.8814" y2="16.1978" width="0.4572" layer="1"/>
-<wire x1="5.4864" y1="18.5928" x2="5.4864" y2="19.3294" width="0.4572" layer="1"/>
-<wire x1="7.8814" y1="16.1978" x2="5.4864" y2="18.5928" width="0.4572" layer="1"/>
-<wire x1="7.8814" y1="7.3794" x2="12.3564" y2="7.3794" width="0.4572" layer="1"/>
-<wire x1="12.3564" y1="7.3794" x2="12.4714" y2="7.2644" width="0.4572" layer="1"/>
-<wire x1="4.8514" y1="7.0794" x2="5.0292" y2="6.9016" width="0.4572" layer="1"/>
-<wire x1="5.0292" y1="6.9016" x2="5.0292" y2="5.334" width="0.4572" layer="1"/>
-<wire x1="5.0292" y1="5.334" x2="5.715" y2="4.6482" width="0.4572" layer="1"/>
+<wire x1="5.4864" y1="18.669" x2="5.4864" y2="19.3294" width="0.4572" layer="1"/>
+<wire x1="5.715" y1="4.6482" x2="4.8514" y2="5.5118" width="0.4572" layer="1"/>
 <wire x1="9.8552" y1="4.6482" x2="12.4714" y2="7.2644" width="0.4572" layer="1"/>
 <wire x1="5.715" y1="4.6482" x2="9.8552" y2="4.6482" width="0.4572" layer="1"/>
@@
 <vertex x="2.667" y="47.3964" curve="-90"/>
 </polygon>
-<wire x1="37.3814" y1="10.6744" x2="37.3814" y2="12.2744" width="0" layer="19" extent="1-1"/>
-<wire x1="7.6764" y1="8.5044" x2="7.7064" y2="8.5344" width="0" layer="19" extent="1-1"/>
+<contactref element="J2" pad="7"/>
+<contactref element="J2" pad="6"/>
+<contactref element="J2" pad="SH1"/>
+<contactref element="J2" pad="SH4"/>
+<contactref element="J2" pad="SH3"/>
+<contactref element="J2" pad="SH2"/>
+<contactref element="J2" pad="5"/>
+<wire x1="4.8514" y1="12.5294" x2="5.3522" y2="13.0302" width="0.4572" layer="1"/>
+<wire x1="5.3522" y1="13.0302" x2="5.9436" y2="13.0302" width="0.4572" layer="1"/>
+<wire x1="4.8514" y1="8.5919" x2="4.6014" y2="8.8419" width="0.1524" layer="1"/>
+<wire x1="4.6014" y1="10.7669" x2="4.6014" y2="12.2794" width="0.8128" layer="1"/>
+<wire x1="4.6014" y1="12.2794" x2="4.8514" y2="12.5294" width="0.1524" layer="1"/>
+<wire x1="4.8514" y1="12.5294" x2="5.4864" y2="13.1644" width="0.1524" layer="1"/>
+<wire x1="5.4864" y1="13.1644" x2="5.4864" y2="18.669" width="0.4572" layer="1"/>
+<wire x1="7.8814" y1="12.2294" x2="7.8814" y2="16.274" width="0.4572" layer="1"/>
+<wire x1="7.8814" y1="16.274" x2="5.4864" y2="18.669" width="0.4572" layer="1"/>
+<wire x1="37.3814" y1="12.2744" x2="39.6814" y2="12.2744" width="0.4572" layer="1"/>
+<wire x1="39.6814" y1="12.2744" x2="41.2814" y2="10.6744" width="0.4572" layer="1"/>
+<wire x1="7.8814" y1="7.3794" x2="10.0464" y2="7.3794" width="0.4572" layer="1"/>
+<wire x1="10.0464" y1="7.3794" x2="11.2014" y2="8.5344" width="0.4572" layer="1"/>
+<wire x1="4.8514" y1="5.5118" x2="4.8514" y2="7.0794" width="0.4572" layer="1"/>
+<wire x1="4.8514" y1="7.0794" x2="4.8514" y2="8.5919" width="0.4572" layer="1"/>
+<wire x1="7.6764" y1="8.5044" x2="11.1714" y2="8.5044" width="0.4572" layer="1"/>
+<wire x1="11.1714" y1="8.5044" x2="11.2014" y2="8.5344" width="0.1524" layer="1"/>
 </signal>
 <signal name="5V">
